File: electronics/kicad/kicad like a pro/4-hands-on-tour-of-kicad-schematic-design/led-torch/led-torch.kicad_sch (KiCad schematic)
At the start: 0 parts

Commit message: done
Other:
- company: (none) -> Digit Lab
- title: (none) -> LED Torch
Changed lines of the file:
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@@
-(kicad_sch (version 20210621) (generator eeschema)
+(kicad_sch (version 20211123) (generator eeschema)
   (paper "A4")
-  (symbol_instances)
+  (title_block
+    (title "LED Torch")
+    (date "2021-11-28")
+    (company "Digit Lab")
+    (comment 1 "Piotr Nowak")
+  )
+  (sheet_instances
+    (path "/" (page "1"))
+  )
 )
