File: electronics/kicad/kicad like a pro/4-hands-on-tour-of-kicad-schematic-design/led-torch/led-torch.kicad_sch (KiCad schematic)
At the start: 0 parts

Commit message: done
Other:
- company: Digit Lab -> eUI Digit Lab
Changed lines of the file:
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@@
     (title "LED Torch")
     (date "2021-11-28")
-    (company "Digit Lab")
+    (company "eUI Digit Lab")
     (comment 1 "Piotr Nowak")
   )

Commit message: done
Parts:
- added BT?: Battery, symbol Device:Battery_Cell
- added D?: LED, symbol Device:LED
- added R?: R, symbol Device:R
- added SW?: SW_DPST_x2, symbol Switch:SW_DPST_x2
Changed lines of the file:
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@@
     (comment 1 "Piotr Nowak")
+  )
+  (symbol (lib_id "Device:Battery_Cell") (at 88.9 104.14 0) (unit 1)
+    (in_bom yes) (on_board yes) (fields_autoplaced)
+    (property "Reference" "BT?" (id 0) (at 92.71 102.4889 0)
+      (effects (font (size 1.27 1.27)) (justify left))
+    )
+    (property "Value" "Battery" (id 1) (at 92.71 105.0289 0)
+      (effects (font (size 1.27 1.27)) (justify left))
+    )
+    (property "Footprint" "" (id 2) (at 88.9 102.616 90)
+      (effects (font (size 1.27 1.27)) hide)
+    )
+    (property "Datasheet" "~" (id 3) (at 88.9 102.616 90)
+      (effects (font (size 1.27 1.27)) hide)
+    )
+    (pin "1")
+    (pin "2")
+  )
+  (symbol (lib_id "Device:LED") (at 72.39 81.28 180) (unit 1)
+    (in_bom yes) (on_board yes) (fields_autoplaced)
+    (property "Reference" "D?" (id 0) (at 73.9775 87.63 0))
+    (property "Value" "LED" (id 1) (at 73.9775 85.09 0))
+    (property "Footprint" "" (id 2) (at 72.39 81.28 0)
+      (effects (font (size 1.27 1.27)) hide)
+    )
+    (property "Datasheet" "~" (id 3) (at 72.39 81.28 0)
+      (effects (font (size 1.27 1.27)) hide)
+    )
+    (pin "1")
+    (pin "2")
+  )
+  (symbol (lib_id "Device:R") (at 88.9 81.28 270) (unit 1)
+    (in_bom yes) (on_board yes) (fields_autoplaced)
+    (property "Reference" "R?" (id 0) (at 88.9 74.93 90))
+    (property "Value" "R" (id 1) (at 88.9 77.47 90))
+    (property "Footprint" "" (id 2) (at 88.9 79.502 90)
+      (effects (font (size 1.27 1.27)) hide)
+    )
+    (property "Datasheet" "~" (id 3) (at 88.9 81.28 0)
+      (effects (font (size 1.27 1.27)) hide)
+    )
+    (pin "1")
+    (pin "2")
+  )
+  (symbol (lib_id "Switch:SW_DPST_x2") (at 106.68 91.44 0) (unit 1)
+    (in_bom yes) (on_board yes) (fields_autoplaced)
+    (property "Reference" "SW?" (id 0) (at 106.68 85.09 0))
+    (property "Value" "SW_DPST_x2" (id 1) (at 106.68 87.63 0))
+    (property "Footprint" "" (id 2) (at 106.68 91.44 0)
+      (effects (font (size 1.27 1.27)) hide)
+    )
+    (property "Datasheet" "~" (id 3) (at 106.68 91.44 0)
+      (effects (font (size 1.27 1.27)) hide)
+    )
+    (pin "1")
+    (pin "2")
   )
   (sheet_instances
     (path "/" (page "1"))
   )
+  (symbol_instances
+    (path "/80925646-d1d5-4a5c-b061-222045730cbf"
+      (reference "BT?") (unit 1) (value "Battery") (footprint "")
+    )
+    (path "/99b7a8c8-7f89-4f97-b2b8-ecdd00b26410"
+      (reference "D?") (unit 1) (value "LED") (footprint "")
+    )
+    (path "/c1778841-bcae-45e9-a3bf-86dd81d61fde"
+      (reference "R?") (unit 1) (value "R") (footprint "")
+    )
+    (path "/ea442210-310a-4326-9aa1-a12310a7108f"
+      (reference "SW?") (unit 1) (value "SW_DPST_x2") (footprint "")
+    )
+  )
 )
