File: electronics/kicad/kicad like a pro/4-hands-on-tour-of-kicad-schematic-design/led-torch2/led-torch2.kicad_sch (KiCad schematic)
At the start: 4 parts, among them SW1 SW_DPST_x2

Commit message: done
Changed lines of the file:
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@@
     (effects (font (size 1 1)) (justify left bottom))
   )
-  (label "bat_pos" (at 127 115.57 270)
+  (label "bat_pos" (at 107.95 112.395 270)
     (effects (font (size 1.27 1.27)) (justify right bottom))
   )
@@
     (effects (font (size 1.27 1.27)) (justify left bottom))
   )
-  (label "LED_anode" (at 107.95 106.68 180)
+  (label "LED_anode" (at 107.95 101.6 180)
     (effects (font (size 1.27 1.27)) (justify right bottom))
   )
