File: electronics/kicad/kicad like a pro/4-hands-on-tour-of-kicad-schematic-design/led-torch2/led-torch2.kicad_pcb (KiCad board)
At the start: 2 copper layers, 4 parts, among them SW1 SW_DPST_x2

Commit message: done
Parts:
- moved D1 23.2 mm to (94.5, 115.1)
- moved SW1 21.6 mm to (117.5, 117.6), turned to 180 degrees
- moved R1 16.8 mm to (101.1, 108.2), turned to 0 degrees
- moved BT1 13.5 mm to (145.8, 107.4), turned to 0 degrees
Other:
- board outline added: 66.3 x 18 mm
Changed lines of the file:
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@@
   (net 4 "Net-(R1-Pad2)")
   (footprint "Button_Switch_THT:SW_TH_Tactile_Omron_B3F-10xx" (layer "F.Cu")
-    (at 124.75 97.23 90)
+    (at 117.55 117.566 180)
     (descr "SW_TH_Tactile_Omron_B3F-10xx_https://www.omron.com/ecb/products/pdf/en-b3f.pdf")
     (tags "Omron B3F-10xx")
@@
     (property "Sheetname" "")
     (attr through_hole)
-    (fp_text reference "SW1" (at 3.25 -2.05 90) (layer "F.SilkS")
-      (effects (font (size 1 1) (thickness 0.15)))
-    )
-    (fp_text value "SW_DPST_x2" (at 3.2 6.5 90) (layer "F.Fab")
-      (effects (font (size 1 1) (thickness 0.15)))
-    )
-    (fp_text user "${REFERENCE}" (at 3.25 2.25 90) (layer "F.Fab")
+    (fp_text reference "SW1" (at 3.25 -2.05) (layer "F.SilkS")
+      (effects (font (size 1 1) (thickness 0.15)))
+    )
+    (fp_text value "SW_DPST_x2" (at 3.2 6.5) (layer "F.Fab")
+      (effects (font (size 1 1) (thickness 0.15)))
+    )
+    (fp_text user "${REFERENCE}" (at 3.25 2.25) (layer "F.Fab")
       (effects (font (size 1 1) (thickness 0.15)))
     )
@@
     (fp_line (start 0.25 -0.75) (end 6.25 -0.75) (layer "F.Fab") (width 0.1))
     (fp_line (start 0.25 5.25) (end 6.25 5.25) (layer "F.Fab") (width 0.1))
-    (pad "1" thru_hole circle locked (at 0 0 90) (size 1.7 1.7) (drill 1) (layers *.Cu *.Mask)
+    (pad "1" thru_hole circle locked (at 0 0 180) (size 1.7 1.7) (drill 1) (layers *.Cu *.Mask)
       (net 4 "Net-(R1-Pad2)") (pinfunction "A") (pintype "passive"))
-    (pad "2" thru_hole circle locked (at 6.5 0 90) (size 1.7 1.7) (drill 1) (layers *.Cu *.Mask)
+    (pad "2" thru_hole circle locked (at 6.5 0 180) (size 1.7 1.7) (drill 1) (layers *.Cu *.Mask)
       (net 2 "Net-(BT1-Pad2)") (pinfunction "B") (pintype "passive"))
-    (pad "3" thru_hole circle locked (at 0 4.5 90) (size 1.7 1.7) (drill 1) (layers *.Cu *.Mask))
-    (pad "4" thru_hole circle locked (at 6.5 4.5 90) (size 1.7 1.7) (drill 1) (layers *.Cu *.Mask))
+    (pad "3" thru_hole circle locked (at 0 4.5 180) (size 1.7 1.7) (drill 1) (layers *.Cu *.Mask))
+    (pad "4" thru_hole circle locked (at 6.5 4.5 180) (size 1.7 1.7) (drill 1) (layers *.Cu *.Mask))
     (model "${KICAD6_3DMODEL_DIR}/Button_Switch_THT.3dshapes/SW_TH_Tactile_Omron_B3F-10xx.wrl"
       (offset (xyz 0 0 0))
@@
   )
   (footprint "Battery:BatteryHolder_Keystone_1058_1x2032" (layer "F.Cu")
-    (at 147.32 93.98 90)
+    (at 145.796 107.442)
     (descr "http://www.keyelco.com/product-pdf.cfm?p=14028")
     (tags "Keystone type 1058 coin cell retainer")
@@
     (property "Sheetname" "")
     (attr smd)
-    (fp_text reference "BT1" (at 0 7.62 90) (layer "F.SilkS")
-      (effects (font (size 1 1) (thickness 0.15)))
-    )
-    (fp_text value "Battery_Cell" (at 0 -9.398 90) (layer "F.Fab")
-      (effects (font (size 1 1) (thickness 0.15)))
-    )
-    (fp_text user "${REFERENCE}" (at 0 0 90) (layer "F.Fab")
+    (fp_text reference "BT1" (at 0 7.62) (layer "F.SilkS")
+      (effects (font (size 1 1) (thickness 0.15)))
+    )
+    (fp_text value "Battery_Cell" (at 0 -9.398) (layer "F.Fab")
+      (effects (font (size 1 1) (thickness 0.15)))
+    )
+    (fp_text user "${REFERENCE}" (at 0 0) (layer "F.Fab")
       (effects (font (size 1 1) (thickness 0.15)))
     )
@@
     (fp_arc (start -10.61275 -3.5) (mid -9.478596 -5.919179) (end -7.802602 -7.999992) (layer "F.Fab") (width 0.1))
     (fp_arc (start -7.802602 7.999992) (mid -9.478596 5.91918) (end -10.61275 3.5) (layer "F.Fab") (width 0.1))
-    (pad "1" smd rect locked (at -14.68 0 90) (size 2.54 3.51) (layers "F.Cu" "F.Paste" "F.Mask")
-      (net 1 "/bat_pos") (pinfunction "+") (pintype "passive"))
-    (pad "2" smd rect locked (at 14.68 0 90) (size 2.54 3.51) (layers "F.Cu" "F.Paste" "F.Mask")
-      (net 2 "Net-(BT1-Pad2)") (pinfunction "-") (pintype "passive"))
+    (pad "1" smd rect locked (at -14.68 0) (size 2.54 3.51) (layers "F.Cu" "F.Paste" "F.Mask")
+      (net 1 "/bat_pos") (pinfunction "+"))
+    (pad "2" smd rect locked (at 14.68 0) (size 2.54 3.51) (layers "F.Cu" "F.Paste" "F.Mask")
+      (net 2 "Net-(BT1-Pad2)") (pinfunction "-"))
     (model "${KICAD6_3DMODEL_DIR}/Battery.3dshapes/BatteryHolder_Keystone_1058_1x2032.wrl"
       (offset (xyz 0 0 0))
@@
   )
   (footprint "Resistor_THT:R_Axial_DIN0204_L3.6mm_D1.6mm_P7.62mm_Horizontal" (layer "F.Cu")
-    (at 114.3 97.79 90)
+    (at 101.092 108.204)
     (descr "Resistor, Axial_DIN0204 series, Axial, Horizontal, pin pitch=7.62mm, 0.167W, length*diameter=3.6*1.6mm^2, http://cdn-reichelt.de/documents/datenblatt/B400/1_4W%23YAG.pdf")
     (tags "Resistor Axial_DIN0204 series Axial Horizontal pin pitch 7.62mm 0.167W length 3.6mm diameter 1.6mm")
@@
     (property "Sheetname" "")
     (attr through_hole)
-    (fp_text reference "R1" (at 3.81 -1.92 90) (layer "F.SilkS")
-      (effects (font (size 1 1) (thickness 0.15)))
-    )
-    (fp_text value "R" (at 3.81 1.92 90) (layer "F.Fab")
-      (effects (font (size 1 1) (thickness 0.15)))
-    )
-    (fp_text user "${REFERENCE}" (at 3.81 0 90) (layer "F.Fab")
+    (fp_text reference "R1" (at 3.81 -1.92) (layer "F.SilkS")
+      (effects (font (size 1 1) (thickness 0.15)))
+    )
+    (fp_text value "R" (at 3.81 1.92) (layer "F.Fab")
+      (effects (font (size 1 1) (thickness 0.15)))
+    )
+    (fp_text user "${REFERENCE}" (at 3.81 0) (layer "F.Fab")
       (effects (font (size 0.72 0.72) (thickness 0.108)))
     )
@@
     (fp_line (start 0 0) (end 2.01 0) (layer "F.Fab") (width 0.1))
     (fp_line (start 5.61 -0.8) (end 2.01 -0.8) (layer "F.Fab") (width 0.1))
-    (pad "1" thru_hole circle locked (at 0 0 90) (size 1.4 1.4) (drill 0.7) (layers *.Cu *.Mask)
+    (pad "1" thru_hole circle locked (at 0 0) (size 1.4 1.4) (drill 0.7) (layers *.Cu *.Mask)
       (net 3 "/LED_cathode") (pintype "passive"))
-    (pad "2" thru_hole oval locked (at 7.62 0 90) (size 1.4 1.4) (drill 0.7) (layers *.Cu *.Mask)
+    (pad "2" thru_hole oval locked (at 7.62 0) (size 1.4 1.4) (drill 0.7) (layers *.Cu *.Mask)
       (net 4 "Net-(R1-Pad2)") (pintype "passive"))
     (model "${KICAD6_3DMODEL_DIR}/Resistor_THT.3dshapes/R_Axial_DIN0204_L3.6mm_D1.6mm_P7.62mm_Horizontal.wrl"
@@
   )
   (footprint "LED_THT:LED_D5.0mm" (layer "F.Cu")
-    (at 104.14 93.98)
+    (at 94.488 115.062)
     (descr "LED, diameter 5.0mm, 2 pins, http://cdn-reichelt.de/documents/datenblatt/A500/LL-504BC2E-009.pdf")
     (tags "LED diameter 5.0mm 2 pins")
@@
     )
   )
+  (gr_line (start 88.646 61.722) (end 88.646 79.756) (layer "Edge.Cuts") (width 0.1))
+  (gr_line (start 154.94 61.722) (end 88.646 61.722) (layer "Edge.Cuts") (width 0.1))
+  (gr_line (start 88.646 79.756) (end 154.94 79.756) (layer "Edge.Cuts") (width 0.1))
+  (gr_circle (center 101.346 70.866) (end 101.346 68.834) (layer "Edge.Cuts") (width 0.1) (fill none))
+  (gr_line (start 154.94 79.756) (end 154.94 61.722) (layer "Edge.Cuts") (width 0.1))
+  (gr_circle (center 101.346 70.866) (end 102.87 69.342) (layer "User.1") (width 0.15) (fill none))
+  (gr_rect (start 88.646 61.823281) (end 154.94 79.756) (layer "User.1") (width 0.15) (fill none))
 )

Commit message: done
Parts:
- moved SW1 49.8 mm to (108.3, 68.6), turned to 0 degrees
- moved D1 45.5 mm to (92.5, 69.6), turned to -90 degrees
- moved BT1 37.5 mm to (137.4, 70.9)
- moved R1 33.6 mm to (98.3, 74.7), turned to 90 degrees
Other:
- outline, holes or cut-outs redrawn
Changed lines of the file:
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@@
   (net 4 "Net-(R1-Pad2)")
   (footprint "Button_Switch_THT:SW_TH_Tactile_Omron_B3F-10xx" (layer "F.Cu")
-    (at 117.55 117.566 180)
+    (at 108.256 68.616)
     (descr "SW_TH_Tactile_Omron_B3F-10xx_https://www.omron.com/ecb/products/pdf/en-b3f.pdf")
     (tags "Omron B3F-10xx")
@@
     (fp_line (start 0.25 -0.75) (end 6.25 -0.75) (layer "F.Fab") (width 0.1))
     (fp_line (start 0.25 5.25) (end 6.25 5.25) (layer "F.Fab") (width 0.1))
-    (pad "1" thru_hole circle locked (at 0 0 180) (size 1.7 1.7) (drill 1) (layers *.Cu *.Mask)
-      (net 4 "Net-(R1-Pad2)") (pinfunction "A") (pintype "passive"))
-    (pad "2" thru_hole circle locked (at 6.5 0 180) (size 1.7 1.7) (drill 1) (layers *.Cu *.Mask)
-      (net 2 "Net-(BT1-Pad2)") (pinfunction "B") (pintype "passive"))
-    (pad "3" thru_hole circle locked (at 0 4.5 180) (size 1.7 1.7) (drill 1) (layers *.Cu *.Mask))
-    (pad "4" thru_hole circle locked (at 6.5 4.5 180) (size 1.7 1.7) (drill 1) (layers *.Cu *.Mask))
+    (pad "1" thru_hole circle locked (at 0 0) (size 1.7 1.7) (drill 1) (layers *.Cu *.Mask)
+      (net 4 "Net-(R1-Pad2)") (pinfunction "A"))
+    (pad "2" thru_hole circle locked (at 6.5 0) (size 1.7 1.7) (drill 1) (layers *.Cu *.Mask)
+      (net 2 "Net-(BT1-Pad2)") (pinfunction "B"))
+    (pad "3" thru_hole circle locked (at 0 4.5) (size 1.7 1.7) (drill 1) (layers *.Cu *.Mask))
+    (pad "4" thru_hole circle locked (at 6.5 4.5) (size 1.7 1.7) (drill 1) (layers *.Cu *.Mask))
     (model "${KICAD6_3DMODEL_DIR}/Button_Switch_THT.3dshapes/SW_TH_Tactile_Omron_B3F-10xx.wrl"
       (offset (xyz 0 0 0))
@@
   )
   (footprint "Battery:BatteryHolder_Keystone_1058_1x2032" (layer "F.Cu")
-    (at 145.796 107.442)
+    (at 137.414 70.866)
     (descr "http://www.keyelco.com/product-pdf.cfm?p=14028")
     (tags "Keystone type 1058 coin cell retainer")
@@
   )
   (footprint "Resistor_THT:R_Axial_DIN0204_L3.6mm_D1.6mm_P7.62mm_Horizontal" (layer "F.Cu")
-    (at 101.092 108.204)
+    (at 98.298 74.676 90)
     (descr "Resistor, Axial_DIN0204 series, Axial, Horizontal, pin pitch=7.62mm, 0.167W, length*diameter=3.6*1.6mm^2, http://cdn-reichelt.de/documents/datenblatt/B400/1_4W%23YAG.pdf")
     (tags "Resistor Axial_DIN0204 series Axial Horizontal pin pitch 7.62mm 0.167W length 3.6mm diameter 1.6mm")
@@
     (property "Sheetname" "")
     (attr through_hole)
-    (fp_text reference "R1" (at 3.81 -1.92) (layer "F.SilkS")
+    (fp_text reference "R1" (at 3.81 -1.92 90) (layer "F.SilkS")
       (effects (font (size 1 1) (thickness 0.15)))
     )
-    (fp_text value "R" (at 3.81 1.92) (layer "F.Fab")
+    (fp_text value "R" (at 3.81 1.92 90) (layer "F.Fab")
       (effects (font (size 1 1) (thickness 0.15)))
     )
-    (fp_text user "${REFERENCE}" (at 3.81 0) (layer "F.Fab")
+    (fp_text user "${REFERENCE}" (at 3.81 0 90) (layer "F.Fab")
       (effects (font (size 0.72 0.72) (thickness 0.108)))
     )
@@
     (fp_line (start 0 0) (end 2.01 0) (layer "F.Fab") (width 0.1))
     (fp_line (start 5.61 -0.8) (end 2.01 -0.8) (layer "F.Fab") (width 0.1))
-    (pad "1" thru_hole circle locked (at 0 0) (size 1.4 1.4) (drill 0.7) (layers *.Cu *.Mask)
-      (net 3 "/LED_cathode") (pintype "passive"))
-    (pad "2" thru_hole oval locked (at 7.62 0) (size 1.4 1.4) (drill 0.7) (layers *.Cu *.Mask)
-      (net 4 "Net-(R1-Pad2)") (pintype "passive"))
+    (pad "1" thru_hole circle locked (at 0 0 90) (size 1.4 1.4) (drill 0.7) (layers *.Cu *.Mask)
+      (net 3 "/LED_cathode"))
+    (pad "2" thru_hole oval locked (at 7.62 0 90) (size 1.4 1.4) (drill 0.7) (layers *.Cu *.Mask)
+      (net 4 "Net-(R1-Pad2)"))
     (model "${KICAD6_3DMODEL_DIR}/Resistor_THT.3dshapes/R_Axial_DIN0204_L3.6mm_D1.6mm_P7.62mm_Horizontal.wrl"
       (offset (xyz 0 0 0))
@@
   )
   (footprint "LED_THT:LED_D5.0mm" (layer "F.Cu")
-    (at 94.488 115.062)
+    (at 92.456 69.591 -90)
     (descr "LED, diameter 5.0mm, 2 pins, http://cdn-reichelt.de/documents/datenblatt/A500/LL-504BC2E-009.pdf")
     (tags "LED diameter 5.0mm 2 pins")
@@
     (property "Sheetname" "")
     (attr through_hole)
-    (fp_text reference "D1" (at 1.27 -3.96) (layer "F.SilkS")
+    (fp_text reference "D1" (at 1.27 -3.96 90) (layer "F.SilkS")
       (effects (font (size 1 1) (thickness 0.15)))
     )
-    (fp_text value "LED" (at 1.27 3.96) (layer "F.Fab")
+    (fp_text value "LED" (at 1.27 3.96 90) (layer "F.Fab")
       (effects (font (size 1 1) (thickness 0.15)))
     )
-    (fp_text user "${REFERENCE}" (at 1.25 0) (layer "F.Fab")
+    (fp_text user "${REFERENCE}" (at 1.25 0 90) (layer "F.Fab")
       (effects (font (size 0.8 0.8) (thickness 0.2)))
     )
@@
     (fp_arc (start -1.23 -1.469694) (mid 4.17 0.000016) (end -1.230016 1.469666) (layer "F.Fab") (width 0.1))
     (fp_circle (center 1.27 0) (end 3.77 0) (layer "F.Fab") (width 0.1) (fill none))
-    (pad "1" thru_hole rect locked (at 0 0) (size 1.8 1.8) (drill 0.9) (layers *.Cu *.Mask)
-      (net 3 "/LED_cathode") (pinfunction "K") (pintype "passive"))
-    (pad "2" thru_hole circle locked (at 2.54 0) (size 1.8 1.8) (drill 0.9) (layers *.Cu *.Mask)
-      (net 1 "/bat_pos") (pinfunction "A") (pintype "passive"))
+    (pad "1" thru_hole rect locked (at 0 0 270) (size 1.8 1.8) (drill 0.9) (layers *.Cu *.Mask)
+      (net 3 "/LED_cathode") (pinfunction "K"))
+    (pad "2" thru_hole circle locked (at 2.54 0 270) (size 1.8 1.8) (drill 0.9) (layers *.Cu *.Mask)
+      (net 1 "/bat_pos") (pinfunction "A"))
     (model "${KICAD6_3DMODEL_DIR}/LED_THT.3dshapes/LED_D5.0mm.wrl"
       (offset (xyz 0 0 0))
@@
     )
   )
-  (gr_line (start 88.646 61.722) (end 88.646 79.756) (layer "Edge.Cuts") (width 0.1))
-  (gr_line (start 154.94 61.722) (end 88.646 61.722) (layer "Edge.Cuts") (width 0.1))
-  (gr_line (start 88.646 79.756) (end 154.94 79.756) (layer "Edge.Cuts") (width 0.1))
-  (gr_circle (center 101.346 70.866) (end 101.346 68.834) (layer "Edge.Cuts") (width 0.1) (fill none))
-  (gr_line (start 154.94 79.756) (end 154.94 61.722) (layer "Edge.Cuts") (width 0.1))
+  (gr_line (start 88.646 61.976) (end 88.646 80.01) (layer "Edge.Cuts") (width 0.1))
+  (gr_line (start 154.94 61.976) (end 88.646 61.976) (layer "Edge.Cuts") (width 0.1))
+  (gr_line (start 88.646 80.01) (end 154.94 80.01) (layer "Edge.Cuts") (width 0.1))
+  (gr_circle (center 103.124 71.12) (end 103.124 69.088) (layer "Edge.Cuts") (width 0.1) (fill none))
+  (gr_line (start 154.94 80.01) (end 154.94 61.976) (layer "Edge.Cuts") (width 0.1))
   (gr_circle (center 101.346 70.866) (end 102.87 69.342) (layer "User.1") (width 0.15) (fill none))
   (gr_rect (start 88.646 61.823281) (end 154.94 79.756) (layer "User.1") (width 0.15) (fill none))

Commit message: done
Parts:
- moved D1 2.80 mm to (92.5, 72.4), turned to 90 degrees
Changed lines of the file:
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@@
   )
   (footprint "LED_THT:LED_D5.0mm" (layer "F.Cu")
-    (at 92.456 69.591 -90)
+    (at 92.456 72.39 90)
     (descr "LED, diameter 5.0mm, 2 pins, http://cdn-reichelt.de/documents/datenblatt/A500/LL-504BC2E-009.pdf")
     (tags "LED diameter 5.0mm 2 pins")
@@
     (fp_arc (start -1.23 -1.469694) (mid 4.17 0.000016) (end -1.230016 1.469666) (layer "F.Fab") (width 0.1))
     (fp_circle (center 1.27 0) (end 3.77 0) (layer "F.Fab") (width 0.1) (fill none))
-    (pad "1" thru_hole rect locked (at 0 0 270) (size 1.8 1.8) (drill 0.9) (layers *.Cu *.Mask)
+    (pad "1" thru_hole rect locked (at 0 0 90) (size 1.8 1.8) (drill 0.9) (layers *.Cu *.Mask)
       (net 3 "/LED_cathode") (pinfunction "K"))
-    (pad "2" thru_hole circle locked (at 2.54 0 270) (size 1.8 1.8) (drill 0.9) (layers *.Cu *.Mask)
+    (pad "2" thru_hole circle locked (at 2.54 0 90) (size 1.8 1.8) (drill 0.9) (layers *.Cu *.Mask)
       (net 1 "/bat_pos") (pinfunction "A"))
     (model "${KICAD6_3DMODEL_DIR}/LED_THT.3dshapes/LED_D5.0mm.wrl"
