File: electronics/kicad/kicad like a pro/4-hands-on-tour-of-kicad-schematic-design/LED torch/LED torch.kicad_sch (KiCad schematic)
At the start: 0 parts

Commit message: done
Parts:
- added BT1: Battery, Battery:BatteryHolder_Keystone_1058_1x2032, symbol Device:Battery_Cell
- added D1: LED, LED_THT:LED_D5.0mm, symbol Device:LED
- added R1: R, Resistor_THT:R_Axial_DIN0204_L3.6mm_D1.6mm_P7.62mm_Horizontal, symbol Device:R
- added SW1: SW_DPST_x2, Button_Switch_THT:SW_TH_Tactile_Omron_B3F-10xx, symbol Switch:SW_DPST_x2
Connections:
- new net: R1.2, SW1.1 (A)
- new net: BT1.1 (+), SW1.2 (B)
- new net: BT1.2 (-), D1.1 (K)
- new net: D1.2 (A), R1.1
Changed lines of the file:
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@@
     (comment 2 "Piotr Nowak")
+  )
+  (wire (pts (xy 109.22 114.3) (xy 109.22 101.6))
+    (stroke (width 0) (type default) (color 0 0 0 0))
+  )
+  (wire (pts (xy 162.56 101.6) (xy 166.37 101.6))
+    (stroke (width 0) (type default) (color 0 0 0 0))
+  )
+  (wire (pts (xy 166.37 114.3) (xy 142.24 114.3))
+    (stroke (width 0) (type default) (color 0 0 0 0))
+  )
+  (wire (pts (xy 166.37 101.6) (xy 166.37 114.3))
+    (stroke (width 0) (type default) (color 0 0 0 0))
+  )
+  (wire (pts (xy 124.46 101.6) (xy 134.62 101.6))
+    (stroke (width 0) (type default) (color 0 0 0 0))
+  )
+  (wire (pts (xy 109.22 101.6) (xy 116.84 101.6))
+    (stroke (width 0) (type default) (color 0 0 0 0))
+  )
+  (wire (pts (xy 134.62 114.3) (xy 109.22 114.3))
+    (stroke (width 0) (type default) (color 0 0 0 0))
+  )
+  (wire (pts (xy 142.24 101.6) (xy 152.4 101.6))
+    (stroke (width 0) (type default) (color 0 0 0 0))
+  )
+  (symbol (lib_id "Switch:SW_DPST_x2") (at 157.48 101.6 0) (unit 1)
+    (in_bom yes) (on_board yes)
+    (property "Reference" "SW1" (id 0) (at 157.48 95.25 0))
+    (property "Value" "SW_DPST_x2" (id 1) (at 157.48 97.79 0))
+    (property "Footprint" "Button_Switch_THT:SW_TH_Tactile_Omron_B3F-10xx" (id 2) (at 158.75 90.17 0)
+      (effects (font (size 0.5 0.5)))
+    )
+    (property "Datasheet" "~" (id 3) (at 157.48 101.6 0)
+      (effects (font (size 0.5 0.5)) hide)
+    )
+    (pin "1")
+    (pin "2")
+    (pin "3")
+    (pin "4")
+  )
+  (symbol (lib_id "Device:Battery_Cell") (at 137.16 114.3 270) (unit 1)
+    (in_bom yes) (on_board yes)
+    (property "Reference" "BT1" (id 0) (at 139.192 107.315 90))
+    (property "Value" "Battery" (id 1) (at 139.192 109.855 90))
+    (property "Footprint" "Battery:BatteryHolder_Keystone_1058_1x2032" (id 2) (at 138.43 105.537 90)
+      (effects (font (size 0.5 0.5)))
+    )
+    (property "Datasheet" "~" (id 3) (at 138.684 114.3 90)
+      (effects (font (size 0.5 0.5)) hide)
+    )
+    (pin "1")
+    (pin "2")
+  )
+  (symbol (lib_id "Device:LED") (at 120.65 101.6 0) (unit 1)
+    (in_bom yes) (on_board yes)
+    (property "Reference" "D1" (id 0) (at 119.0625 95.25 0))
+    (property "Value" "LED" (id 1) (at 119.0625 97.79 0))
+    (property "Footprint" "LED_THT:LED_D5.0mm" (id 2) (at 119.761 90.932 0)
+      (effects (font (size 0.5 0.5)))
+    )
+    (property "Datasheet" "~" (id 3) (at 120.65 101.6 0)
+      (effects (font (size 0.5 0.5)) hide)
+    )
+    (pin "1")
+    (pin "2")
+  )
+  (symbol (lib_id "Device:R") (at 138.43 101.6 90) (unit 1)
+    (in_bom yes) (on_board yes)
+    (property "Reference" "R1" (id 0) (at 138.43 95.25 90))
+    (property "Value" "R" (id 1) (at 138.43 97.79 90))
+    (property "Footprint" "Resistor_THT:R_Axial_DIN0204_L3.6mm_D1.6mm_P7.62mm_Horizontal" (id 2) (at 140.97 92.71 90)
+      (effects (font (size 0.5 0.5)))
+    )
+    (property "Datasheet" "~" (id 3) (at 138.43 101.6 0)
+      (effects (font (size 0.5 0.5)) hide)
+    )
+    (pin "1")
+    (pin "2")
   )
   (sheet_instances
     (path "/" (page "1"))
   )
+  (symbol_instances
+    (path "/4228a43c-d16f-498b-b303-cb0e38244f2d"
+      (reference "BT1") (unit 1) (value "Battery") (footprint "Battery:BatteryHolder_Keystone_1058_1x2032")
+    )
+    (path "/949ec1ea-25bf-4883-bfdb-7c233d317c8e"
+      (reference "D1") (unit 1) (value "LED") (footprint "LED_THT:LED_D5.0mm")
+    )
+    (path "/9a76052a-7ad6-4560-a2ff-80e0dbba13a0"
+      (reference "R1") (unit 1) (value "R") (footprint "Resistor_THT:R_Axial_DIN0204_L3.6mm_D1.6mm_P7.62mm_Horizontal")
+    )
+    (path "/19c0985e-a2e2-428d-8568-45996498bc67"
+      (reference "SW1") (unit 1) (value "SW_DPST_x2") (footprint "Button_Switch_THT:SW_TH_Tactile_Omron_B3F-10xx")
+    )
+  )
 )
