File: electronics/kicad/kicad like a pro/4-hands-on-tour-of-kicad-schematic-design/LED torch/LED torch.kicad_pcb (KiCad board)
At the start: 2 copper layers, 73.7 x 17.8 mm, 4 parts, among them SW1 SW_DPST_x2

Commit message: done
Other:
- board size 73.7 x 17.8 mm -> 76.8 x 25.1 mm
Changed lines of the file:
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@@
     )
   )
-  (gr_rect (start 111.76 88.9) (end 185.42 106.68) (layer "Edge.Cuts") (width 0.1) (fill none))
+  (gr_line (start 177.710297 90.301831) (end 184.983974 90.290014) (layer "Edge.Cuts") (width 0.1))
+  (gr_arc (start 115.57 105.156) (mid 108.204 97.79) (end 115.57 90.424) (layer "Edge.Cuts") (width 0.1))
+  (gr_line (start 185.031307 105.152668) (end 177.8 105.156) (layer "Edge.Cuts") (width 0.1))
+  (gr_line (start 184.983974 90.290014) (end 185.031307 105.152668) (layer "Edge.Cuts") (width 0.1))
+  (gr_arc (start 177.8 105.156) (mid 167.64 110.339245) (end 157.48 105.156) (layer "Edge.Cuts") (width 0.1))
+  (gr_line (start 115.57 90.424) (end 157.48 90.424) (layer "Edge.Cuts") (width 0.1))
+  (gr_arc (start 157.48 90.424) (mid 167.564218 85.240984) (end 177.710297 90.301831) (layer "Edge.Cuts") (width 0.1))
+  (gr_line (start 115.57 105.156) (end 157.48 105.156) (layer "Edge.Cuts") (width 0.1))
   (gr_circle (center 147.32 97.79) (end 146.05 97.79) (layer "Edge.Cuts") (width 0.1) (fill none))
   (gr_circle (center 129.54 97.79) (end 128.27 97.79) (layer "Edge.Cuts") (width 0.1) (fill none))
-  (gr_circle (center 143.51 121.92) (end 146.05 121.92) (layer "User.1") (width 0.15) (fill none))
-  (gr_rect (start 129.54 113.03) (end 195.58 130.81) (layer "User.1") (width 0.15) (fill none))
+  (gr_circle (center 167.64 97.79) (end 167.894 85.344) (layer "User.1") (width 0.15) (fill none))
   (segment (start 141.68 98.837919) (end 143.51 97.007919) (width 0.25) (layer "F.Cu") (net 1))
   (segment (start 143.51 97.007919) (end 143.51 95.25) (width 0.25) (layer "F.Cu") (net 1))

Commit message: done
Parts:
- added REF**: KiCad-Logo_8mm_SilkScreen, Symbol:KiCad-Logo_8mm_SilkScreen, B.Cu at (167.6, 97.5)
Other:
- board text added: "+"
- board text added: "-"
- board text added: "v1.0.0"
