File: electronics/kicad/kicad like a pro/8-fundamentals-symbols-and-eeschema/8-fundamentals-symbols-and-eeschema.kicad_pcb (KiCad board)
At the start: 2 copper layers, 2 parts, among them J1 6P6C_Shielded, U1 ATmega328PB-A

Commit message: done
Parts:
- removed U1: ATmega328PB-A, Package_QFP:TQFP-32_7x7mm_P0.8mm
- added J2: Conn_01x01_Female, Connector_Pin:Pin_D0.7mm_L6.5mm_W1.8mm_FlatFork, F.Cu at (134.6, 91.4)
- added J3: Conn_01x01_Female, Connector_Pin:Pin_D0.7mm_L6.5mm_W1.8mm_FlatFork, F.Cu at (134.6, 99.1)
- added J4: Conn_01x01_Female, Connector_Pin:Pin_D0.7mm_L6.5mm_W1.8mm_FlatFork, F.Cu at (154.9, 99.1)
- added R1: R, Resistor_THT:R_Axial_DIN0207_L6.3mm_D2.5mm_P7.62mm_Horizontal, F.Cu at (132.1, 81.3)
- added R2: R, Resistor_SMD:R_0603_1608Metric_Pad0.98x0.95mm_HandSolder, F.Cu at (121.8, 92.3)
- added U2: NA555_PN, Package_DIP:DIP-8_W7.62mm, F.Cu at (116.8, 76.2)
- J1: value 6P6C_Shielded -> Conn_01x01_Female; footprint Connector_Audio:Jack_XLR-6.35mm_Neutrik_NCJ6FI-H-0_Horizontal -> Connector_Pin:Pin_D0.7mm_L6.5mm_W1.8mm_FlatFork
- moved J1 26.2 mm to (154.9, 91.4)
Connections:
- J1 pad 1: unconnected-(J1-Pad1) -> /net_1

Commit message: done
Parts:
- added R3: R, Resistor_THT:R_Axial_DIN0207_L6.3mm_D2.5mm_P7.62mm_Horizontal, F.Cu at (168.9, 68.6)
- added R4: R, Resistor_SMD:R_0603_1608Metric_Pad0.98x0.95mm_HandSolder, F.Cu at (158.7, 79.6)
- added R5: R, Resistor_THT:R_Axial_DIN0207_L6.3mm_D2.5mm_P7.62mm_Horizontal, F.Cu at (186.9, 68.6)
- added R6: R, Resistor_SMD:R_0603_1608Metric_Pad0.98x0.95mm_HandSolder, F.Cu at (187.5, 74.9)
- added U1: NA555_PN, Package_DIP:DIP-8_W7.62mm, F.Cu at (158.1, 68.6)
- added U3: Test, Capacitor_SMD:CP_Elec_3x5.4, F.Cu at (190.5, 86.4)
- moved R2 15.3 mm to (134.6, 83.8), turned to 180 degrees
- moved R1 6.35 mm to (137.2, 77.5), turned to 90 degrees
- moved U2 3.80 mm to (116.8, 72.4)
Connections:
- J3 pad 1: /net_1 -> Global_1
- J4 pad 1: /net_1 -> Global_1
- U2 pad 2: unconnected-(U2-Pad2) -> /Sheet 2/hier_1_label
Routing:
- net Global_1: track 0.00 -> 89.4 mm
- net /net_2: track 0.00 -> 29.3 mm
- net /Sheet 2/Sheet 3/hier_a: track 0.00 -> 20.4 mm, vias 0 -> 2
- net Net-(R2-Pad2): track 0.00 -> 19.5 mm
- net Net-(R1-Pad1): track 0.00 -> 7.02 mm
