File: electronics/kicad/kicad like a pro/8-fundamentals-symbols-and-eeschema/8-fundamentals-symbols-and-eeschema.kicad_sch (KiCad schematic)
At the start: 2 parts, among them J1 6P6C_Shielded, U1 ATmega328PB-A

Commit message: done
Parts:
- removed J1: 6P6C_Shielded, Connector_Audio:Jack_XLR-6.35mm_Neutrik_NCJ6FI-H-0_Horizontal, symbol Connector:6P6C_Shielded
- removed U1: ATmega328PB-A, Package_QFP:TQFP-32_7x7mm_P0.8mm, symbol MCU_Microchip_ATmega:ATmega328PB-A
- added J1, J2, J3, J4: Conn_01x01_Female, Connector_Pin:Pin_D0.7mm_L6.5mm_W1.8mm_FlatFork, symbol Connector:Conn_01x01_Female
- added R1: R, Resistor_THT:R_Axial_DIN0207_L6.3mm_D2.5mm_P7.62mm_Horizontal, symbol Device:R
- added R2: R, Resistor_SMD:R_0603_1608Metric_Pad0.98x0.95mm_HandSolder, symbol Device:R
- added U2: NA555_PN, Package_DIP:DIP-8_W7.62mm, symbol Peters_Library:NA555_PN
Connections:
- new net: R1.1, R2.1
- new net: R2.2, U2.3 (OUT)
- new net net_1: J1.1 (Pin_1), J2.1 (Pin_1), J3.1 (Pin_1), J4.1 (Pin_1)
- new net net_2: R1.2, U2.5 (CONT)
Changed lines of the file:
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@@
 (kicad_sch (version 20211123) (generator eeschema)
   (paper "A4")
-  (symbol (lib_id "Connector:6P6C_Shielded") (at 160.02 91.44 0) (unit 1)
-    (in_bom yes) (on_board yes)
-    (property "Reference" "J1" (id 0) (at 160.02 76.2 0))
-    (property "Value" "6P6C_Shielded" (id 1) (at 160.02 78.74 0))
-    (property "Footprint" "Connector_Audio:Jack_XLR-6.35mm_Neutrik_NCJ6FI-H-0_Horizontal" (id 2) (at 165.1 72.39 0))
-    (property "Datasheet" "~" (id 3) (at 160.02 90.805 90)
+  (wire (pts (xy 212.09 92.71) (xy 205.74 92.71))
+    (stroke (width 0) (type default) (color 0 0 0 0))
+  )
+  (wire (pts (xy 185.42 100.33) (xy 185.42 118.11))
+    (stroke (width 0) (type default) (color 0 0 0 0))
+  )
+  (wire (pts (xy 29.21 33.02) (xy 55.88 33.02))
+    (stroke (width 0) (type default) (color 0 0 0 0))
+  )
+  (wire (pts (xy 160.02 129.54) (xy 212.09 129.54))
+    (stroke (width 0) (type default) (color 0 0 0 0))
+  )
+  (wire (pts (xy 152.4 118.11) (xy 146.05 118.11))
+    (stroke (width 0) (type default) (color 0 0 0 0))
+  )
+  (wire (pts (xy 146.05 129.54) (xy 152.4 129.54))
+    (stroke (width 0) (type default) (color 0 0 0 0))
+  )
+  (wire (pts (xy 146.05 118.11) (xy 146.05 129.54))
+    (stroke (width 0) (type default) (color 0 0 0 0))
+  )
+  (wire (pts (xy 185.42 118.11) (xy 160.02 118.11))
+    (stroke (width 0) (type default) (color 0 0 0 0))
+  )
+  (wire (pts (xy 212.09 129.54) (xy 212.09 92.71))
+    (stroke (width 0) (type default) (color 0 0 0 0))
+  )
+  (wire (pts (xy 29.21 25.4) (xy 55.88 25.4))
+    (stroke (width 0) (type default) (color 0 0 0 0))
+  )
+  (label "net_1" (at 40.64 33.02 0)
+    (effects (font (size 1.27 1.27)) (justify left bottom))
+  )
+  (label "net_2" (at 171.45 118.11 0)
+    (effects (font (size 1.27 1.27)) (justify left bottom))
+  )
+  (label "net_1" (at 40.64 25.4 0)
+    (effects (font (size 1.27 1.27)) (justify left bottom))
+  )
+  (symbol (lib_id "Device:R") (at 156.21 129.54 90) (unit 1)
+    (in_bom yes) (on_board yes) (fields_autoplaced)
+    (property "Reference" "R2" (id 0) (at 156.21 123.19 90))
+    (property "Value" "R" (id 1) (at 156.21 125.73 90))
+    (property "Footprint" "Resistor_SMD:R_0603_1608Metric_Pad0.98x0.95mm_HandSolder" (id 2) (at 156.21 131.318 90)
       (effects (font (size 1.27 1.27)) hide)
     )
-    (property "Custom Field" "frergeger" (id 4) (at 158.75 105.41 0))
+    (property "Datasheet" "~" (id 3) (at 156.21 129.54 0)
+      (effects (font (size 1.27 1.27)) hide)
+    )
+    (pin "1")
+    (pin "2")
+  )
+  (symbol (lib_id "Connector:Conn_01x01_Female") (at 24.13 33.02 180) (unit 1)
+    (in_bom yes) (on_board yes) (fields_autoplaced)
+    (property "Reference" "J3" (id 0) (at 24.765 27.94 0))
+    (property "Value" "Conn_01x01_Female" (id 1) (at 24.765 30.48 0))
+    (property "Footprint" "Connector_Pin:Pin_D0.7mm_L6.5mm_W1.8mm_FlatFork" (id 2) (at 24.13 33.02 0)
+      (effects (font (size 1.27 1.27)) hide)
+    )
+    (property "Datasheet" "~" (id 3) (at 24.13 33.02 0)
+      (effects (font (size 1.27 1.27)) hide)
+    )
+    (pin "1")
+  )
+  (symbol (lib_id "Connector:Conn_01x01_Female") (at 60.96 25.4 0) (unit 1)
+    (in_bom yes) (on_board yes) (fields_autoplaced)
+    (property "Reference" "J2" (id 0) (at 62.23 24.1299 0)
+      (effects (font (size 1.27 1.27)) (justify left))
+    )
+    (property "Value" "Conn_01x01_Female" (id 1) (at 62.23 26.6699 0)
+      (effects (font (size 1.27 1.27)) (justify left))
+    )
+    (property "Footprint" "Connector_Pin:Pin_D0.7mm_L6.5mm_W1.8mm_FlatFork" (id 2) (at 60.96 25.4 0)
+      (effects (font (size 1.27 1.27)) hide)
+    )
+    (property "Datasheet" "~" (id 3) (at 60.96 25.4 0)
+      (effects (font (size 1.27 1.27)) hide)
+    )
+    (pin "1")
+  )
+  (symbol (lib_id "Connector:Conn_01x01_Female") (at 24.13 25.4 180) (unit 1)
+    (in_bom yes) (on_board yes) (fields_autoplaced)
+    (property "Reference" "J1" (id 0) (at 24.765 20.32 0))
+    (property "Value" "Conn_01x01_Female" (id 1) (at 24.765 22.86 0))
+    (property "Footprint" "Connector_Pin:Pin_D0.7mm_L6.5mm_W1.8mm_FlatFork" (id 2) (at 24.13 25.4 0)
+      (effects (font (size 1.27 1.27)) hide)
+    )
+    (property "Datasheet" "~" (id 3) (at 24.13 25.4 0)
+      (effects (font (size 1.27 1.27)) hide)
+    )
+    (pin "1")
+  )
+  (symbol (lib_id "Device:R") (at 156.21 118.11 90) (unit 1)
+    (in_bom yes) (on_board yes) (fields_autoplaced)
+    (property "Reference" "R1" (id 0) (at 156.21 111.76 90))
+    (property "Value" "R" (id 1) (at 156.21 114.3 90))
+    (property "Footprint" "Resistor_THT:R_Axial_DIN0207_L6.3mm_D2.5mm_P7.62mm_Horizontal" (id 2) (at 156.21 119.888 90)
+      (effects (font (size 1.27 1.27)) hide)
+    )
+    (property "Datasheet" "~" (id 3) (at 156.21 118.11 0)
+      (effects (font (size 1.27 1.27)) hide)
+    )
+    (pin "1")
+    (pin "2")
+  )
+  (symbol (lib_id "Connector:Conn_01x01_Female") (at 60.96 33.02 0) (unit 1)
+    (in_bom yes) (on_board yes) (fields_autoplaced)
+    (property "Reference" "J4" (id 0) (at 62.23 31.7499 0)
+      (effects (font (size 1.27 1.27)) (justify left))
+    )
+    (property "Value" "Conn_01x01_Female" (id 1) (at 62.23 34.2899 0)
+      (effects (font (size 1.27 1.27)) (justify left))
+    )
+    (property "Footprint" "Connector_Pin:Pin_D0.7mm_L6.5mm_W1.8mm_FlatFork" (id 2) (at 60.96 33.02 0)
+      (effects (font (size 1.27 1.27)) hide)
+    )
+    (property "Datasheet" "~" (id 3) (at 60.96 33.02 0)
+      (effects (font (size 1.27 1.27)) hide)
+    )
+    (pin "1")
+  )
+  (symbol (lib_id "Peters_Library:NA555_PN") (at 194.31 81.28 0) (unit 1)
+    (in_bom yes) (on_board yes) (fields_autoplaced)
+    (property "Reference" "U2" (id 0) (at 197.5994 78.74 0)
+      (effects (font (size 1.27 1.27)) (justify left))
+    )
+    (property "Value" "NA555_PN" (id 1) (at 197.5994 81.28 0)
+      (effects (font (size 1.27 1.27)) (justify left))
+    )
+    (property "Footprint" "Package_DIP:DIP-8_W7.62mm" (id 2) (at 198.12 69.85 0)
+      (effects (font (size 1.27 1.27)) hide)
+    )
+    (property "Datasheet" "https://www.ti.com/lit/ds/symlink/ne555.pdf" (id 3) (at 200.66 66.04 0)
+      (effects (font (size 1.27 1.27)) hide)
+    )
     (pin "1")
     (pin "2")
@@
     (pin "5")
     (pin "6")
-    (pin "SH")
-  )
-  (symbol (lib_id "MCU_Microchip_ATmega:ATmega328PB-A") (at 110.49 91.44 0) (unit 1)
-    (in_bom yes) (on_board yes)
-    (property "Reference" "U1" (id 0) (at 112.5094 129.54 0)
-      (effects (font (size 1.27 1.27)) (justify left))
-    )
-    (property "Value" "ATmega328PB-A" (id 1) (at 112.5094 132.08 0)
-      (effects (font (size 1.27 1.27)) (justify left))
-    )
-    (property "Footprint" "Package_QFP:TQFP-32_7x7mm_P0.8mm" (id 2) (at 110.49 135.89 0)
-      (effects (font (size 1.27 1.27) italic))
-    )
-    (property "Datasheet" "http://ww1.microchip.com/downloads/en/DeviceDoc/40001906C.pdf" (id 3) (at 110.49 91.44 0)
-      (effects (font (size 1.27 1.27)) hide)
-    )
-    (pin "1")
-    (pin "10")
-    (pin "11")
-    (pin "12")
-    (pin "13")
-    (pin "14")
-    (pin "15")
-    (pin "16")
-    (pin "17")
-    (pin "18")
-    (pin "19")
-    (pin "2")
-    (pin "20")
-    (pin "21")
-    (pin "22")
-    (pin "23")
-    (pin "24")
-    (pin "25")
-    (pin "26")
-    (pin "27")
-    (pin "28")
-    (pin "29")
-    (pin "3")
-    (pin "30")
-    (pin "31")
-    (pin "32")
-    (pin "4")
-    (pin "5")
-    (pin "6")
     (pin "7")
     (pin "8")
-    (pin "9")
   )
   (sheet_instances
@@
   )
   (symbol_instances
-    (path "/cce4fcb6-5758-488f-94a4-ac5a136900a9"
-      (reference "J1") (unit 1) (value "6P6C_Shielded") (footprint "Connector_Audio:Jack_XLR-6.35mm_Neutrik_NCJ6FI-H-0_Horizontal")
+    (path "/6017f552-93c3-4633-80dd-f32df2051afb"
+      (reference "J1") (unit 1) (value "Conn_01x01_Female") (footprint "Connector_Pin:Pin_D0.7mm_L6.5mm_W1.8mm_FlatFork")
     )
-    (path "/f30071c0-1232-482f-8694-7ee43e366144"
-      (reference "U1") (unit 1) (value "ATmega328PB-A") (footprint "Package_QFP:TQFP-32_7x7mm_P0.8mm")
+    (path "/4c296fc9-6b9f-4b23-b823-99742664e100"
+      (reference "J2") (unit 1) (value "Conn_01x01_Female") (footprint "Connector_Pin:Pin_D0.7mm_L6.5mm_W1.8mm_FlatFork")
+    )
+    (path "/30319230-1a29-4327-8796-6f01749a6efa"
+      (reference "J3") (unit 1) (value "Conn_01x01_Female") (footprint "Connector_Pin:Pin_D0.7mm_L6.5mm_W1.8mm_FlatFork")
+    )
+    (path "/be844d2a-ff7f-45af-990a-a178587cbef0"
+      (reference "J4") (unit 1) (value "Conn_01x01_Female") (footprint "Connector_Pin:Pin_D0.7mm_L6.5mm_W1.8mm_FlatFork")
+    )
+    (path "/81f75093-56e5-4864-8056-f0c48a7e765c"
+      (reference "R1") (unit 1) (value "R") (footprint "Resistor_THT:R_Axial_DIN0207_L6.3mm_D2.5mm_P7.62mm_Horizontal")
+    )
+    (path "/0cf54d67-fcbf-48d0-9699-6801b5a03fc0"
+      (reference "R2") (unit 1) (value "R") (footprint "Resistor_SMD:R_0603_1608Metric_Pad0.98x0.95mm_HandSolder")
+    )
+    (path "/cd99df50-7aef-40dc-aca4-73982397dd93"
+      (reference "U2") (unit 1) (value "NA555_PN") (footprint "Package_DIP:DIP-8_W7.62mm")
     )
   )

Commit message: done
Parts:
- added U3: Test, Capacitor_SMD:CP_Elec_3x5.4, symbol Peters_Library:Test
Connections:
- net net_1: no longer J3.1 (Pin_1), J4.1 (Pin_1)
- net Sheet 2/hier_1_label: now reaches U2.2 (TRIG)
- new net Gbl_1: J3.1 (Pin_1), J4.1 (Pin_1)
- new net Sheet 2/hier_2_label: U3.1 (Input)
- no-connect marks 0 -> 6
Other:
- added sheet Sheet 2 (sub-sheet.kicad_sch)
Changed lines of the file:
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@@
 (kicad_sch (version 20211123) (generator eeschema)
   (paper "A4")
+  (junction (at 40.64 33.02) (diameter 0) (color 0 0 0 0)
+  )
+  (no_connect (at 195.58 81.28))
+  (no_connect (at 185.42 88.9))
+  (no_connect (at 185.42 92.71))
+  (no_connect (at 205.74 88.9))
+  (no_connect (at 195.58 107.95))
+  (no_connect (at 167.64 50.8))
   (wire (pts (xy 212.09 92.71) (xy 205.74 92.71))
     (stroke (width 0) (type default) (color 0 0 0 0))
   )
+  (wire (pts (xy 167.64 35.56) (xy 160.02 35.56))
+    (stroke (width 0) (type default) (color 0 0 0 0))
+  )
   (wire (pts (xy 185.42 100.33) (xy 185.42 118.11))
     (stroke (width 0) (type default) (color 0 0 0 0))
   )
-  (wire (pts (xy 29.21 33.02) (xy 55.88 33.02))
+  (wire (pts (xy 120.65 34.29) (xy 120.65 62.23))
+    (stroke (width 0) (type default) (color 0 0 0 0))
+  )
+  (wire (pts (xy 29.21 33.02) (xy 40.64 33.02))
+    (stroke (width 0) (type default) (color 0 0 0 0))
+  )
+  (wire (pts (xy 40.64 33.02) (xy 40.64 41.91))
     (stroke (width 0) (type default) (color 0 0 0 0))
   )
@@
     (stroke (width 0) (type default) (color 0 0 0 0))
   )
+  (wire (pts (xy 120.65 62.23) (xy 146.05 62.23))
+    (stroke (width 0) (type default) (color 0 0 0 0))
+  )
+  (wire (pts (xy 40.64 33.02) (xy 55.88 33.02))
+    (stroke (width 0) (type default) (color 0 0 0 0))
+  )
   (wire (pts (xy 152.4 118.11) (xy 146.05 118.11))
     (stroke (width 0) (type default) (color 0 0 0 0))
   )
+  (wire (pts (xy 146.05 43.18) (xy 167.64 43.18))
+    (stroke (width 0) (type default) (color 0 0 0 0))
+  )
   (wire (pts (xy 146.05 129.54) (xy 152.4 129.54))
     (stroke (width 0) (type default) (color 0 0 0 0))
   )
+  (wire (pts (xy 160.02 35.56) (xy 160.02 96.52))
+    (stroke (width 0) (type default) (color 0 0 0 0))
+  )
+  (wire (pts (xy 146.05 62.23) (xy 146.05 43.18))
+    (stroke (width 0) (type default) (color 0 0 0 0))
+  )
   (wire (pts (xy 146.05 118.11) (xy 146.05 129.54))
     (stroke (width 0) (type default) (color 0 0 0 0))
@@
     (stroke (width 0) (type default) (color 0 0 0 0))
   )
+  (wire (pts (xy 160.02 96.52) (xy 185.42 96.52))
+    (stroke (width 0) (type default) (color 0 0 0 0))
+  )
   (wire (pts (xy 29.21 25.4) (xy 55.88 25.4))
     (stroke (width 0) (type default) (color 0 0 0 0))
-  )
-  (label "net_1" (at 40.64 33.02 0)
-    (effects (font (size 1.27 1.27)) (justify left bottom))
   )
   (label "net_2" (at 171.45 118.11 0)
@@
   (label "net_1" (at 40.64 25.4 0)
     (effects (font (size 1.27 1.27)) (justify left bottom))
+  )
+  (global_label "Gbl_1" (shape input) (at 40.64 41.91 270) (fields_autoplaced)
+    (effects (font (size 1.27 1.27)) (justify right))
+    (property "Intersheet References" "${INTERSHEET_REFS}" (id 0) (at 40.7194 52.5479 90)
+      (effects (font (size 1.27 1.27)) (justify right) hide)
+    )
   )
   (symbol (lib_id "Device:R") (at 156.21 129.54 90) (unit 1)
@@
     )
     (property "Datasheet" "~" (id 3) (at 24.13 33.02 0)
+      (effects (font (size 1.27 1.27)) hide)
+    )
+    (pin "1")
+  )
+  (symbol (lib_id "Peters_Library:Test") (at 123.19 31.75 0) (unit 1)
+    (in_bom yes) (on_board yes) (fields_autoplaced)
+    (property "Reference" "U3" (id 0) (at 134.62 38.7349 0)
+      (effects (font (size 1.27 1.27)) (justify left))
+    )
+    (property "Value" "Test" (id 1) (at 134.62 41.2749 0)
+      (effects (font (size 1.27 1.27)) (justify left))
+    )
+    (property "Footprint" "Capacitor_SMD:CP_Elec_3x5.4" (id 2) (at 127 29.21 0)
+      (effects (font (size 1.27 1.27)) hide)
+    )
+    (property "Datasheet" "" (id 3) (at 127 29.21 0)
       (effects (font (size 1.27 1.27)) hide)
     )
@@
     (pin "8")
   )
+  (sheet (at 167.64 30.48) (size 55.88 38.1) (fields_autoplaced)
+    (stroke (width 0.1524) (type solid) (color 0 0 0 0))
+    (fill (color 0 0 0 0.0000))
+    (property "Sheet name" "Sheet 2" (id 0) (at 167.64 29.7684 0)
+      (effects (font (size 1.27 1.27)) (justify left bottom))
+    )
+    (property "Sheet file" "sub-sheet.kicad_sch" (id 1) (at 167.64 69.1646 0)
+      (effects (font (size 1.27 1.27)) (justify left top))
+    )
+    (pin "hier_1_label" input (at 167.64 35.56 180)
+      (effects (font (size 1.27 1.27)) (justify left))
+    )
+    (pin "hier_2_label" input (at 167.64 43.18 180)
+      (effects (font (size 1.27 1.27)) (justify left))
+    )
+    (pin "hier_3_label" input (at 167.64 50.8 180)
+      (effects (font (size 1.27 1.27)) (justify left))
+    )
+  )
   (sheet_instances
     (path "/" (page "1"))
+    (path "/93a2ae69-e835-460b-b7d2-bea765cbeae8" (page "2"))
+    (path "/93a2ae69-e835-460b-b7d2-bea765cbeae8/8bff1114-85b5-4e01-b3d3-4e5ce7680f93" (page "3"))
   )
   (symbol_instances
@@
       (reference "R2") (unit 1) (value "R") (footprint "Resistor_SMD:R_0603_1608Metric_Pad0.98x0.95mm_HandSolder")
     )
+    (path "/93a2ae69-e835-460b-b7d2-bea765cbeae8/5281fa9b-ae5a-4a6d-9571-5503aac8f06b"
+      (reference "R3") (unit 1) (value "R") (footprint "Resistor_THT:R_Axial_DIN0207_L6.3mm_D2.5mm_P7.62mm_Horizontal")
+    )
+    (path "/93a2ae69-e835-460b-b7d2-bea765cbeae8/e8805821-17d1-4bb7-92c3-3e62d7252073"
+      (reference "R4") (unit 1) (value "R") (footprint "Resistor_SMD:R_0603_1608Metric_Pad0.98x0.95mm_HandSolder")
+    )
+    (path "/93a2ae69-e835-460b-b7d2-bea765cbeae8/8bff1114-85b5-4e01-b3d3-4e5ce7680f93/677a00dd-ef08-4682-94e7-068c2dac3d3a"
+      (reference "R5") (unit 1) (value "R") (footprint "Resistor_THT:R_Axial_DIN0207_L6.3mm_D2.5mm_P7.62mm_Horizontal")
+    )
+    (path "/93a2ae69-e835-460b-b7d2-bea765cbeae8/8bff1114-85b5-4e01-b3d3-4e5ce7680f93/e8417a0d-f393-41aa-8a4c-319d4df1da09"
+      (reference "R6") (unit 1) (value "R") (footprint "Resistor_SMD:R_0603_1608Metric_Pad0.98x0.95mm_HandSolder")
+    )
+    (path "/93a2ae69-e835-460b-b7d2-bea765cbeae8/5cdbc076-d610-45b3-b76f-226c34860bd4"
+      (reference "U1") (unit 1) (value "NA555_PN") (footprint "Package_DIP:DIP-8_W7.62mm")
+    )
     (path "/cd99df50-7aef-40dc-aca4-73982397dd93"
       (reference "U2") (unit 1) (value "NA555_PN") (footprint "Package_DIP:DIP-8_W7.62mm")
     )
-  )
+    (path "/3ba79e01-b82f-435f-94c6-5a349c4616a4"
+      (reference "U3") (unit 1) (value "Test") (footprint "Capacitor_SMD:CP_Elec_3x5.4")
+    )
+  )
