File: electronics/kicad/kicad like a pro/9-footprints-and-pcbnew/_autosave-BreadboardPowerSupply_v2.kicad_pcb (KiCad board)
At the start: 2 copper layers, 30.1 x 52.2 mm, 19 parts, among them J1 Barrel_Jack_Switch, J2 Conn_02x02_Odd_Even, J3 Conn_02x02_Odd_Even, SW1 SW_DPDT_x2, U1 LM7805_TO220

Commit message: done
Parts:
- C1: value CP -> CP.
Connections:
- J1 pad 3: Net-(J1-Pad3) -> unconnected-(J1-Pad3)
- SW1 pad 3: Net-(SW1-Pad3) -> unconnected-(SW1-Pad3)
