File: electronics/kicad/kicad like a pro/9-footprints-and-pcbnew/_autosave-BreadboardPowerSupply_v2.kicad_sch (KiCad schematic)
At the start: 15 parts, among them J1 Barrel_Jack_Switch, J2 Conn_02x02_Odd_Even, J3 Conn_02x02_Odd_Even, SW1 SW_DPDT_x2, U1 LM7805_TO220

Commit message: done
Parts:
- C1: value CP -> CP.
Changed lines of the file:
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@@
       (effects (font (size 1.27 1.27)) (justify left))
     )
-    (property "Value" "CP" (id 1) (at 116.0272 91.313 0)
+    (property "Value" "CP." (id 1) (at 116.0272 91.313 0)
       (effects (font (size 1.27 1.27)) (justify left))
     )
@@
     )
     (path "/00000000-0000-0000-0000-00005b9f5330"
-      (reference "C1") (unit 1) (value "CP") (footprint "Capacitor_THT:CP_Radial_D10.0mm_P5.00mm")
+      (reference "C1") (unit 1) (value "CP.") (footprint "Capacitor_THT:CP_Radial_D10.0mm_P5.00mm")
     )
     (path "/00000000-0000-0000-0000-00005b9f55af"
