File: electronics/kicad/kicad like a pro/10-simple-brteadboard-pwr-supply/10-simple-brteadboard-pwr-supply.kicad_sch (KiCad schematic)
At the start: 0 parts

Commit message: done
Parts:
- added C1: 10u, Capacitor_THT:C_Disc_D3.0mm_W1.6mm_P2.50mm, symbol Device:C
- added C2: 0.1u, Capacitor_THT:C_Disc_D3.0mm_W1.6mm_P2.50mm, symbol Device:C
- added C3: 1u, Capacitor_THT:C_Disc_D3.0mm_W1.6mm_P2.50mm, symbol Device:C
- added D1: LED, LED_THT:LED_D5.0mm, symbol Device:LED
- added J1: Barrel_Jack_Switch, Connector_BarrelJack:BarrelJack_Horizontal, symbol Connector:Barrel_Jack_Switch
- added J2, J5: Conn_01x03_Male, Connector_PinHeader_2.54mm:PinHeader_1x03_P2.54mm_Vertical, symbol Connector:Conn_01x03_Male
- added J3, J6: Conn_01x02_Male, Connector_PinHeader_2.54mm:PinHeader_1x02_P2.54mm_Vertical, symbol Connector:Conn_01x02_Male
- added J4, J7: Screw_Terminal_01x02, TerminalBlock:TerminalBlock_bornier-2_P5.08mm, symbol Connector:Screw_Terminal_01x02
- added R1, R2: 330, Resistor_THT:R_Axial_DIN0204_L3.6mm_D1.6mm_P7.62mm_Horizontal, symbol Device:R
- added R3: 560, Resistor_THT:R_Axial_DIN0204_L3.6mm_D1.6mm_P7.62mm_Horizontal, symbol Device:R
- added S1: EG1218, digikey-footprints:Switch_Slide_11.6x4mm_EG1218, symbol dk_Slide-Switches:EG1218
- added U1: LM317_TO-220, Package_TO_SOT_THT:TO-220-3_Vertical, symbol Regulator_Linear:LM317_TO-220
- added U2: LM7805_TO220, Package_TO_SOT_THT:TO-220-3_Vertical, symbol Regulator_Linear:LM7805_TO220
Other:
- company: (none) -> Domisoft
- title: (none) -> Learning KiCad with a simple project

Commit message: done
Connections:
- net at R2.1: now also R3.2, U1.1 (ADJ)
- net 3.3V: now reaches R2.2
- net 3.3V: now also C3.1, J2.1 (Pin_1), J5.1 (Pin_1), U1.2 (VO)
- net GND: now reaches C3.2
- net GND: now also C1.2, C2.2, D1.1 (K), J1.2, J1.3, J3.1 (Pin_1), J4.1 (Pin_1), J6.1 (Pin_1), J7.1 (Pin_1), R3.1, U2.2 (GND)
- net at R1.1: now also D1.2 (A)
- net 12V: now reaches R1.2
- net 12V: now also C1.1, S1.1, U1.3 (VI), U2.1 (VI)
- net at J4.2 (Pin_2): now also J2.2 (Pin_2), J3.2 (Pin_2)
- net 5V: now reaches J2.3 (Pin_3)
- net 5V: now also C2.1, J5.3 (Pin_3), U2.3 (VO)
- net at J1.1: now also S1.2
- net at J7.2 (Pin_2): now also J5.2 (Pin_2), J6.2 (Pin_2)
- no-connect marks 0 -> 1
Other:
- moved on the sheet: C1, C2, C3, D1, J2, J3, J4, J5, J6, J7, R1, R2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
